Commit message: Cover Xacro include and parameter project layout [skip ci]

File: tests/fixtures/local-assistant/robot.urdf.xacro (robot description, xacro)
@@ -2,12 +2,7 @@
 <robot name="test_robot" xmlns:xacro="http://www.ros.org/wiki/xacro">
   <xacro:arg name="joint_name" default="elbow"/>
+  <xacro:include filename="parts/joint.xacro"/>
   <link name="base"/>
   <link name="arm"/>
-  <joint name="$(arg joint_name)" type="revolute">
-    <parent link="base"/>
-    <child link="arm"/>
-    <origin xyz="0 0 0" rpy="0 0 0"/>
-    <axis xyz="0 0 1"/>
-    <limit lower="-1" upper="1" effort="1" velocity="1"/>
-  </joint>
+  <xacro:arm_joint name="$(arg joint_name)"/>
 </robot>
